File: rgb565-experiment.sch (KiCad schematic (older format))
At the start: 6 parts, among them J1 ST_SHIFTER_SOCKET, U1 74HC00, U2 ST_SHIFTER, U3 ST_SHIFTER, U4 74HC245, U5 74HC245

Commit message: schematic complete with color dac
Parts:
- added C1, C2, C3, C4, C5, C6: 0.1uF, symbol Device:C
- added R? (x3): 1K2, symbol Device:R_US
- added R? (x3): 2K4, symbol Device:R_US
- added R? (x3): 4K7, symbol Device:R_US
- added R? (x3): 9K1, symbol Device:R_US
- added R? (x3): 20K, symbol Device:R_US
- added R? (x3): 39K, symbol Device:R_US
- added SW1: SW_SPDT, symbol Switch:SW_SPDT
- added U5: 74LS257, symbol 74xx:74LS257
- renumbered U5 to U6
Connections:
- net r0 is gone; now on net r1: U3.29 (R0)
- net a5: now also U5.3 (I1a), U5.5 (I0b); no longer U4.19 (CE)
- net b0: now also R?.1; no longer U3.23 (B0)
- net b1: now also U3.23 (B0), R?.1; no longer U2.23 (B0)
- net b2: now also U3.22 (B1), R?.1; no longer U2.22 (B1)
- net b3: now also U2.23 (B0), R?.1; no longer U2.21 (B2)
- net b4: now also U2.22 (B1), R?.1; no longer U3.22 (B1)
- net g0: now also R?.1
- net g1: now also U3.25 (G1), R?.1; no longer U2.26 (G0)
- net g2: now also U3.24 (G2), R?.1; no longer U2.25 (G1)
- net g3: now also U2.26 (G0), R?.1; no longer U2.24 (G2)
- net g4: now also U2.25 (G1), R?.1; no longer U3.25 (G1)
- net g5: now also U2.24 (G2), R?.1; no longer U3.24 (G2)
- net gnd: now also C1.2, C2.2, C3.2, C4.2, C5.2, C6.2, SW1.3 (C), U5.10 (I1d), U5.11 (I0d), U5.13 (I1c), U5.14 (I0c), U5.15 (OE), U5.8 (GND)
- net r1: now also R?.1; no longer U2.29 (R0)
- net r2: now also U3.28 (R1), R?.1; no longer U2.28 (R1)
- net r3: now also U2.29 (R0), R?.1; no longer U2.27 (R2)
- net r4: now also U2.28 (R1), R?.1; no longer U3.28 (R1)
- net vcc: now also C1.1, C2.1, C3.1, C4.1, C5.1, C6.1, SW1.1 (A), U5.16 (VCC)
- net blue: now reaches J1.21 (B2)
- net blue: now also R?.2, R?.2, R?.2, R?.2, R?.2, R?.2
- net green: now reaches J1.24 (G2)
- net green: now also R?.2, R?.2, R?.2, R?.2, R?.2, R?.2
- net red: now reaches J1.27 (R2)
- net red: now also R?.2, R?.2, R?.2, R?.2, R?.2, R?.2
- net at U1.8: now also U5.2 (I0a), U5.6 (I1b); no longer U6.19 (CE)
- new net: SW1.2 (B), U5.1 (S)
- new net: U4.19 (CE), U5.4 (Za)
- new net: U5.7 (Zb), U6.19 (CE)
- new net b5: R?.1, U2.21 (B2)
- new net r5: R?.1, R?.1, U2.27 (R2)
- no-connect marks 15 -> 14
Other:
- note added: "Assume that address\nof palette registers \nis 0xxxx"
- note added: "Assume that address\nof palette registers \nis 1xxxx"
- note added: "Auxiliary shifter"
- note added: "Main Shifter"
- note added: "Maybe, instead of two 74x245,\njust use two 74x257 ?\nBecause in my mod, the auxiliary\nshifter is only allowed to\nreceive data from the bus.\n"
- note added: "The original mod state to use one 74x243 + one 74x245.\nI don't know how it is done\n\nI used two 74x245, and use a5 to select wich one to \nenable. I assume that address 0 to 15 are the palette\nregisters. It may be wrong.\n\nThe 74x257 allow to test whether the palette registers\nare in the range 0—15 or 16—31"
- note added: "«Additionally, jumpers are installed across \neach of three 3.6K ohm resistors on the motherboard. \nThese resistors are easily traced from the Shifter \nsocket pins 21, 24, and 27.» \n(From the original text)\n"
- note removed: "TODO : \n* bypass capacitor\n* resistor ladder to analog R,V,B signal"
- note removed: "The original mod state to use one 74x243 + one 74x245.\nI don't know how it is done\n\nI used two 74x245, and use a5 to select wich one to \nenable. I assume that address 0 to 15 are the palette\nregisters. It may be wrong.\n\nTODO : plan a way to swap the selection logic for testing."
- moved on the sheet: J1, U1A, U1B, U1C, U1D, U1E, U2, U3, U4, U6
