File: rgb565-experiment.kicad_pcb (KiCad board)
At the start: 4 copper layers, 101.6 x 71.1 mm, 34 parts, among them J1 ST_SHIFTER_SOCKET, J2 Conn_01x02, SW1 SW_SPDT, U1 74HC00, U2 ST_SHIFTER, U3 ST_SHIFTER, U4 74HC245, U5 74LS257, U6 74HC245

Commit message: almost done routing
Parts:
- moved C1 24.1 mm to (166.4, 127.0), turned to 270 degrees
- moved U1 18.2 mm to (170.2, 130.8), turned to 90 degrees
- moved U4 2.54 mm to (170.2, 105.4)
- moved C3 2.54 mm to (156.2, 82.5)
- moved C4 2.54 mm to (166.4, 101.6)
- moved C5 1.27 mm to (190.5, 114.3)
- moved U5 1.27 mm to (186.7, 110.5)
- moved C6 0.38 mm to (165.1, 88.5)
Connections:
- U1 pad 3: Net-(U1-Pad12) -> Net-(U1-Pad13)
- U1 pad 6: Net-(U1-Pad13) -> Net-(U1-Pad12)
Routing:
- net /d15: track 45.1 -> 142.8 mm, vias 0 -> 1
- net /d12: track 45.1 -> 142.5 mm, vias 0 -> 1
- net /d13: track 45.1 -> 140.8 mm, vias 0 -> 1
- net /d14: track 45.1 -> 136.3 mm, vias 0 -> 1
- net /d11: track 45.1 -> 131.8 mm, vias 0 -> 1
- net /d7: track 45.1 -> 117.0 mm, vias 0 -> 2
- net /d3: track 45.1 -> 111.3 mm, vias 0 -> 2
- net /cs2: track 0.00 -> 58.2 mm
- net /d8: track 20.8 -> 76.9 mm, vias 0 -> 1
- net /d9: track 20.8 -> 76.5 mm, vias 0 -> 1
- net /rxw: track 20.8 -> 74.8 mm, vias 0 -> 1
- net /d5: track 20.8 -> 70.0 mm, vias 0 -> 1
- net /d4: track 20.8 -> 70.0 mm, vias 0 -> 1
- net /d6: track 20.8 -> 70.0 mm, vias 0 -> 1
- net /d0: track 20.8 -> 65.9 mm, vias 0 -> 1
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
Commit message: done initial routing
Routing:
- net /rxw: track 74.8 -> 99.5 mm
- net /a3: track 20.8 -> 45.2 mm
- net /a2: track 20.8 -> 45.1 mm
- net /a4: track 20.8 -> 45.1 mm
- net /a1: track 20.8 -> 45.1 mm
- net /a5: track 96.5 -> 120.7 mm
